File: hardware/gpsclock/gpsclock.kicad_sch (KiCad schematic)
At the start: 142 parts, among them J1 USB-C power, J2 u.FL (active antenna), J3 SWD, J4 UART debug, Q1 phototransistor (TBD), SW1 Brightness, U1 STM32G030F6P6, U11 74HCT595, U12 74HCT595, U13 74HCT595, U14 74HCT595, U15 74HCT595, U16 74HCT595, U17 74HCT595, U18 74HCT595, U19 74HCT595, U2 AP2112K-3.3, U3 ATGM336H-5N31, Y1 16MHz CMOS 3.3V

Commit message: Apply schematic review fixes
Multi-agent review of rev 0.1 (19 findings, 7 confirmed):
- U2 regulator had no footprint: generator now falls back to the library
  default, and check_netlist.py fails on parts without a footprint
- F1 750 mA hold; correct the 5 V current figures (74 LEDs, not 72)
- 33R series resistors R100/R101 on SR_CLK and SR_LATCH
- Cut VBUS bulk capacitance toward the USB 10 uF sink limit
- Antenna feed per ATGM336H-5N manual 2.7.1: R8 now 0R
- BOM reference designators regenerated from the netlist

Co-Authored-By: Claude Opus 5.5 <noreply@anthropic.com>
Claude-Session: https://claude.ai/code/session_01XvyGkgyfnJ274YR57krtzr
Parts:
- removed C21: 10u, Capacitor_SMD:C_0805_2012Metric, symbol Device:C
- added R100, R101: 33, Resistor_SMD:R_0603_1608Metric, symbol Device:R
- C1: value 10u -> 4.7u
- F1: value 500mA hold -> 750mA hold
- R8: value 10 -> 0
- U2: footprint (none) -> Package_TO_SOT_SMD:SOT-23-5
Connections:
- net SR_CLK: now also R100.2; no longer U1.12 (PA5)
- net SR_LATCH: now also R101.2; no longer U1.15 (PB0/PB1/PB2/PA8)
- new net SR_CLK_MCU: R100.1, U1.12 (PA5)
- new net SR_LATCH_MCU: R101.1, U1.15 (PB0/PB1/PB2/PA8)
Other:
- note added: "All 74 LEDs on: ~0.42-0.47 A from 5 V. Firmware must cap /OE duty for an all-segments self-test."
- note added: "Segment resistors 470R: ~5.7-6.4 mA per LED. 8 LEDs per 595 (~46-51 mA); U12/U14 drive 9 (~51-58 mA). Limit 70 mA."
- note removed: "Segment resistors 470R: (5 V - ~2.0 V LED - ~0.3 V drop) / 470 = ~5.7 mA per segment, <= 46 mA per 595."

Commit message: Rev 0.2: five DC56-11 duals (HH:MM:SS.mmmm), mode button, firmware plan
- Display: ten digits on five Kingbright DC56-11 18-pin duals, tenth
  74HCT595 (U20); pin mapping from the KiCad library symbol
- SW2 mode button on PC15; refs renumbered (R120/R121, C21, C11-C20)
- docs/firmware-features.md: modes, seconds-alive epoch with leap
  seconds, buttons, settings
- BOM and shopping lists updated for the duals (~$2.13-3.65 each)

Co-Authored-By: Claude Opus 5.5 <noreply@anthropic.com>
Claude-Session: https://claude.ai/code/session_01XvyGkgyfnJ274YR57krtzr
Parts:
- removed DS6, DS7, DS8, DS9: 0.56in CC red, Display_7Segment:7SegmentLED_LTS6760_LTS6780, symbol gpsclock:7SEG_CC_5161AS
- removed R100: 33, Resistor_SMD:R_0603_1608Metric, symbol Device:R
- added C21: 10u, Capacitor_SMD:C_0805_2012Metric, symbol Device:C
- added R102, R103, R104, R105, R106, R107, R108: 470, Resistor_SMD:R_0603_1608Metric, symbol Device:R
- added R120, R121: 33, Resistor_SMD:R_0603_1608Metric, symbol Device:R
- added SW2: Mode, Button_Switch_THT:SW_PUSH_6mm, symbol Switch:SW_Push
- added U20: 74HCT595, Package_SO:SOIC-16_3.9x9.9mm_P1.27mm, symbol 74xx:74HCT595
- C20: value 10u -> 100n; footprint Capacitor_SMD:C_0805_2012Metric -> Capacitor_SMD:C_0603_1608Metric
- DS1, DS2, DS3, DS4, DS5: value 0.56in CC red -> DC56-11EWA; footprint Display_7Segment:7SegmentLED_LTS6760_LTS6780 -> Display_7Segment:DA56-11SURKWA; symbol gpsclock:7SEG_CC_5161AS -> Display_Character:DC56-11EWA
- R101: value 33 -> 470
Connections:
- net +5V: now also C21.1, U20.10 (~{SRCLR}), U20.16 (VCC)
- net D1_A: now also DS1.16 (DIG1_A); no longer DS1.7 (A)
- net D1_B: now also DS1.15 (DIG1_B); no longer DS1.6 (B)
- net D1_C: now also DS1.3 (DIG1_C); no longer DS1.4 (C)
- net D1_DP: now also DS1.4 (DP1); no longer DS1.5 (DP)
- net D1_F: now also DS1.18 (DIG1_F); no longer DS1.9 (F)
- net D1_G: now also DS1.17 (DIG1_G); no longer DS1.10 (G)
- net D2_A: now also DS1.11 (DIG2_A); no longer DS2.7 (A)
- net D2_B: now also DS1.10 (DIG2_B); no longer DS2.6 (B)
- net D2_C: now also DS1.8 (DIG2_C); no longer DS2.4 (C)
- net D2_D: now also DS1.6 (DIG2_D); no longer DS2.2 (D)
- net D2_E: now also DS1.5 (DIG2_E); no longer DS2.1 (E)
- net D2_F: now also DS1.12 (DIG2_F); no longer DS2.9 (F)
- net D2_G: now also DS1.7 (DIG2_G); no longer DS2.10 (G)
- net D3_A: now also DS2.16 (DIG1_A); no longer DS3.7 (A)
- net D3_B: now also DS2.15 (DIG1_B); no longer DS3.6 (B)
- net D3_C: now also DS2.3 (DIG1_C); no longer DS3.4 (C)
- net D3_D: now also DS2.2 (DIG1_D); no longer DS3.2 (D)
- net D3_DP: now also DS2.4 (DP1); no longer DS3.5 (DP)
- net D3_E: now also DS2.1 (DIG1_E); no longer DS3.1 (E)
- net D3_F: now also DS2.18 (DIG1_F); no longer DS3.9 (F)
- net D3_G: now also DS2.17 (DIG1_G); no longer DS3.10 (G)
- net D4_A: now also DS2.11 (DIG2_A); no longer DS4.7 (A)
- net D4_B: now also DS2.10 (DIG2_B); no longer DS4.6 (B)
- net D4_C: now also DS2.8 (DIG2_C); no longer DS4.4 (C)
- net D4_D: now also DS2.6 (DIG2_D); no longer DS4.2 (D)
- net D4_E: now also DS2.5 (DIG2_E); no longer DS4.1 (E)
- net D4_F: now also DS2.12 (DIG2_F); no longer DS4.9 (F)
- net D4_G: now also DS2.7 (DIG2_G); no longer DS4.10 (G)
- net D5_A: now also DS3.16 (DIG1_A); no longer DS5.7 (A)
- net D5_B: now also DS3.15 (DIG1_B); no longer DS5.6 (B)
- net D5_C: now also DS3.3 (DIG1_C); no longer DS5.4 (C)
- net D5_D: now also DS3.2 (DIG1_D); no longer DS5.2 (D)
- net D5_DP: now also DS3.4 (DP1); no longer DS5.5 (DP)
- net D5_E: now also DS3.1 (DIG1_E); no longer DS5.1 (E)
- net D5_F: now also DS3.18 (DIG1_F); no longer DS5.9 (F)
- net D5_G: now also DS3.17 (DIG1_G); no longer DS5.10 (G)
- net D6_A: now also DS3.11 (DIG2_A)
- net D6_B: now also DS3.10 (DIG2_B)
- net D6_C: now also DS3.8 (DIG2_C)
- net D6_D: now also DS3.6 (DIG2_D)
- net D6_DP: now also DS3.9 (DP2)
- net D6_E: now also DS3.5 (DIG2_E)
- net D6_F: now also DS3.12 (DIG2_F)
- net D6_G: now also DS3.7 (DIG2_G)
- net D7_A: now also DS4.16 (DIG1_A)
- net D7_B: now also DS4.15 (DIG1_B)
- net D7_C: now also DS4.3 (DIG1_C)
- net D7_D: now also DS4.2 (DIG1_D)
- net D7_DP: now also DS4.4 (DP1)
- net D7_E: now also DS4.1 (DIG1_E)
- net D7_F: now also DS4.18 (DIG1_F)
- net D7_G: now also DS4.17 (DIG1_G)
- net D8_A: now also DS4.11 (DIG2_A)
- net D8_B: now also DS4.10 (DIG2_B)
- net D8_C: now also DS4.8 (DIG2_C)
- net D8_D: now also DS4.6 (DIG2_D)
- net D8_DP: now also DS4.9 (DP2)
- net D8_E: now also DS4.5 (DIG2_E)
- net D8_F: now also DS4.12 (DIG2_F)
- net D8_G: now also DS4.7 (DIG2_G)
- net D9_A: now also DS5.16 (DIG1_A)
- net D9_B: now also DS5.15 (DIG1_B)
- net D9_C: now also DS5.3 (DIG1_C)
- net D9_D: now also DS5.2 (DIG1_D)
- net D9_DP: now also DS5.4 (DP1)
- net D9_E: now also DS5.1 (DIG1_E)
- net D9_F: now also DS5.18 (DIG1_F)
- net D9_G: now also DS5.17 (DIG1_G)
- net DISP_OE: now also U20.13 (~{OE})
- net GND: now also DS1.13 (DIG2_CC), DS1.14 (DIG1_CC), DS2.13 (DIG2_CC), DS2.14 (DIG1_CC), DS3.13 (DIG2_CC), DS3.14 (DIG1_CC), DS4.13 (DIG2_CC), DS4.14 (DIG1_CC), DS5.13 (DIG2_CC), DS5.14 (DIG1_CC), C21.2, SW2.2, U20.8 (GND); no longer DS1.3 (CC), DS1.8 (CC), DS2.3 (CC), DS2.8 (CC), DS3.3 (CC), DS3.8 (CC), DS4.3 (CC), DS4.8 (CC), DS5.3 (CC), DS5.8 (CC)
- net SR_CLK: now also R120.2, U20.11 (SRCLK)
- net SR_CLK_MCU: now also R120.1
- net SR_LATCH: now also R121.2, U20.12 (RCLK); no longer R101.2
- net SR_LATCH_MCU: now also R121.1; no longer R101.1
- net BTN_MODE: now reaches U1.3 (PC15)
- net BTN_MODE: now also SW2.1
- net SR_D10: now reaches U19.9 (QH')
- net SR_D10: now also U20.14 (SER)
- net BTN renamed BTN_BRIGHT
- new net D10_A: DS5.11 (DIG2_A), R101.2
- new net D10_B: DS5.10 (DIG2_B), R102.2
- new net D10_C: DS5.8 (DIG2_C), R103.2
- new net D10_D: DS5.6 (DIG2_D), R104.2
- new net D10_DP: DS5.9 (DP2), R108.2
- new net D10_E: DS5.5 (DIG2_E), R105.2
- new net D10_F: DS5.12 (DIG2_F), R106.2
- new net D10_G: DS5.7 (DIG2_G), R107.2
- new net D10_QA: R101.1, U20.15 (QA)
- new net D10_QB: R102.1, U20.1 (QB)
- new net D10_QC: R103.1, U20.2 (QC)
- new net D10_QD: R104.1, U20.3 (QD)
- new net D10_QE: R105.1, U20.4 (QE)
- new net D10_QF: R106.1, U20.5 (QF)
- new net D10_QG: R107.1, U20.6 (QG)
- new net D10_QH: R108.1, U20.7 (QH)
- no-connect marks 11 -> 10
Other:
- note added: "All 82 LEDs on: ~0.47-0.52 A from 5 V. Firmware must cap /OE duty for an all-segments self-test."
- note added: "Chain: SR_DATA -> U11 -> U12 ... -> U20. All latch together on SR_LATCH. /OE = PWM brightness."
- note added: "Colons: between DS1|DS2 (COL1) and DS2|DS3 (COL2). Two 3 mm red LEDs each, driven from QH of U12 / U14."
- note added: "DISPLAY: HH:MM:SS.mmmm, 10 digits on five Kingbright DC56-11 duals, each digit statically driven by a 74HCT595 (5 V)."
- note added: "Digit 10: 1/10000 s (DS5 DIG2)"
- note added: "Digit 1: H tens (DS1 DIG1)"
- note added: "Digit 2: H units (DS1 DIG2)"
- note added: "Digit 3: M tens (DS2 DIG1)"
- note added: "Digit 4: M units (DS2 DIG2)"
- note added: "Digit 5: S tens (DS3 DIG1)"
- note added: "Digit 6: S units, DP = decimal point (DS3 DIG2)"
- note added: "Digit 7: 1/10 s (DS4 DIG1)"
- note added: "Digit 8: 1/100 s (DS4 DIG2)"
- note added: "Digit 9: 1/1000 s (DS5 DIG1)"
- note added: "Displays: Kingbright DC56-11EWA, 0.56in dual digit, common cathode, 18 pins (every segment on its own pin)."
- note added: "I/O: SWD, debug UART, mode + brightness buttons, status LED, light sensor (optional)"
- note removed: "All 74 LEDs on: ~0.42-0.47 A from 5 V. Firmware must cap /OE duty for an all-segments self-test."
- note removed: "Chain: SR_DATA -> U11 -> U12 ... -> U19. All latch together on SR_LATCH. /OE = PWM brightness."
- note removed: "Colons: between DS2|DS3 (COL1) and DS4|DS5 (COL2). Two 3 mm red LEDs each, driven from QH of U12 / U14."
- note removed: "DISPLAY: HH:MM:SS.mmm, 9 digits, each statically driven by a 74HCT595 (5 V)."
- note removed: "DS1: H tens"
- note removed: "DS2: H units"
- note removed: "DS3: M tens"
- note removed: "DS4: M units"
- note removed: "DS5: S tens"
- note removed: "DS6: S units (DP = decimal point)"
- note removed: "DS7: 1/10 s"
- note removed: "DS8: 1/100 s"
- note removed: "DS9: 1/1000 s"
- note removed: "I/O: SWD, debug UART, button, status LED, light sensor (optional)"
- moved on the sheet: C10, C11, C12, C13, C14, C15, C16, C17, C18, C19, C20, Q1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
